File: pcbs/tinker/classical_guitar/classical_guitar_fretboard.sch (KiCad schematic (older format))
At the start: 167 parts, among them U1 AT42QT1110-A, U2 AT42QT1110-A, U3 AT42QT1110-A

Commit message: Rearranged schematic again and establishing pcb layout
Parts:
- added H1, H2, H3, H4: MountingHole_Pad, MountingHole:MountingHole_4.3mm_M4_Pad_Via, symbol Mechanical:MountingHole_Pad
- Cd1, Cd2, Cd3, Cd4, Cd5, Cd6: footprint (none) -> Capacitor_SMD:C_0402_1005Metric_Pad0.74x0.62mm_HandSolder
- Cs1: renamed from Cs11; footprint (none) -> Capacitor_SMD:C_0603_1608Metric_Pad1.08x0.95mm_HandSolder
- Cs10: renamed from Cs20; footprint (none) -> Capacitor_SMD:C_0603_1608Metric_Pad1.08x0.95mm_HandSolder
- Cs11: renamed from Cs21; footprint (none) -> Capacitor_SMD:C_0603_1608Metric_Pad1.08x0.95mm_HandSolder
- Cs12: renamed from Cs22; footprint (none) -> Capacitor_SMD:C_0603_1608Metric_Pad1.08x0.95mm_HandSolder
- Cs13: renamed from Cs23; footprint (none) -> Capacitor_SMD:C_0603_1608Metric_Pad1.08x0.95mm_HandSolder
- Cs14: renamed from Cs24; footprint (none) -> Capacitor_SMD:C_0603_1608Metric_Pad1.08x0.95mm_HandSolder
- Cs15: renamed from Cs25; footprint (none) -> Capacitor_SMD:C_0603_1608Metric_Pad1.08x0.95mm_HandSolder
- Cs16: renamed from Cs26; footprint (none) -> Capacitor_SMD:C_0603_1608Metric_Pad1.08x0.95mm_HandSolder
- Cs17: renamed from Cs27; footprint (none) -> Capacitor_SMD:C_0603_1608Metric_Pad1.08x0.95mm_HandSolder
- Cs18: renamed from Cs28; footprint (none) -> Capacitor_SMD:C_0603_1608Metric_Pad1.08x0.95mm_HandSolder
- Cs19: renamed from Cs29; footprint (none) -> Capacitor_SMD:C_0603_1608Metric_Pad1.08x0.95mm_HandSolder
- Cs2: renamed from Cs12; footprint (none) -> Capacitor_SMD:C_0603_1608Metric_Pad1.08x0.95mm_HandSolder
- Cs20: renamed from Cs30; footprint (none) -> Capacitor_SMD:C_0603_1608Metric_Pad1.08x0.95mm_HandSolder
- Cs21: renamed from Cs1; footprint (none) -> Capacitor_SMD:C_0603_1608Metric_Pad1.08x0.95mm_HandSolder
- Cs22: renamed from Cs2; footprint (none) -> Capacitor_SMD:C_0603_1608Metric_Pad1.08x0.95mm_HandSolder
- Cs23: renamed from Cs3; footprint (none) -> Capacitor_SMD:C_0603_1608Metric_Pad1.08x0.95mm_HandSolder
- Cs24: renamed from Cs4; footprint (none) -> Capacitor_SMD:C_0603_1608Metric_Pad1.08x0.95mm_HandSolder
- Cs25: renamed from Cs5; footprint (none) -> Capacitor_SMD:C_0603_1608Metric_Pad1.08x0.95mm_HandSolder
- Cs26: renamed from Cs6; footprint (none) -> Capacitor_SMD:C_0603_1608Metric_Pad1.08x0.95mm_HandSolder
- Cs27: renamed from Cs7; footprint (none) -> Capacitor_SMD:C_0603_1608Metric_Pad1.08x0.95mm_HandSolder
- Cs28: renamed from Cs8; footprint (none) -> Capacitor_SMD:C_0603_1608Metric_Pad1.08x0.95mm_HandSolder
- Cs29: renamed from Cs9; footprint (none) -> Capacitor_SMD:C_0603_1608Metric_Pad1.08x0.95mm_HandSolder
- Cs3: renamed from Cs13; footprint (none) -> Capacitor_SMD:C_0603_1608Metric_Pad1.08x0.95mm_HandSolder
- Cs30: renamed from Cs10; footprint (none) -> Capacitor_SMD:C_0603_1608Metric_Pad1.08x0.95mm_HandSolder
- Cs4: renamed from Cs14; footprint (none) -> Capacitor_SMD:C_0603_1608Metric_Pad1.08x0.95mm_HandSolder
- Cs5: renamed from Cs15; footprint (none) -> Capacitor_SMD:C_0603_1608Metric_Pad1.08x0.95mm_HandSolder
- Cs6: renamed from Cs16; footprint (none) -> Capacitor_SMD:C_0603_1608Metric_Pad1.08x0.95mm_HandSolder
- Cs7: renamed from Cs17; footprint (none) -> Capacitor_SMD:C_0603_1608Metric_Pad1.08x0.95mm_HandSolder
- Cs8: renamed from Cs18; footprint (none) -> Capacitor_SMD:C_0603_1608Metric_Pad1.08x0.95mm_HandSolder
- Cs9: renamed from Cs19; footprint (none) -> Capacitor_SMD:C_0603_1608Metric_Pad1.08x0.95mm_HandSolder
- E1, E10, E11, E12, E13, E14, E15, E16, E17, E18, E19, E2, E20, E21, E22, E23, E24, E25, E26, E27, E28, E29, E3, E30, E4, E5, E6, E7, E8, E9: footprint (none) -> Custom_Electrode:Circle_10mm
- JPch1, JPch2, JPch3, JPe1, JPe10, JPe11, JPe12, JPe13, JPe14, JPe15, JPe16, JPe17, JPe18, JPe19, JPe2, JPe20, JPe21, JPe22, JPe23, JPe24, JPe25, JPe26, JPe27, JPe28, JPe29, JPe3, JPe30, JPe4, JPe5, JPe6, JPe7, JPe8, JPe9, JPmiso1, JPmiso2, JPmiso3, JPmosi1, JPmosi2, JPmosi3, JPsck1, JPsck2, JPsck3: footprint (none) -> Jumper:SolderJumper-3_P1.3mm_Bridged12_RoundedPad1.0x1.5mm_NumberLabels
- Rch1, Rs1, Rs10, Rs11, Rs12, Rs13, Rs14, Rs15, Rs16, Rs17, Rs18, Rs19, Rs2, Rs20, Rs21, Rs22, Rs23, Rs24, Rs25, Rs26, Rs27, Rs28, Rs29, Rs3, Rs30, Rs31, Rs32, Rs33, Rs34, Rs35, Rs36, Rs37, Rs38, Rs39, Rs4, Rs5, Rs6, Rs7, Rs8, Rs9: footprint (none) -> Resistor_SMD:R_0603_1608Metric_Pad0.98x0.95mm_HandSolder
- U1, U2, U3: footprint Package:TQFP-32_7.0x7.0mm_P0.8mm -> Package_QFP:TQFP-32_7x7mm_P0.8mm
Connections:
- net C_MISO: now also JPmiso1.2 (C), JPmiso2.2 (C), JPmiso3.2 (C); no longer JPmiso1.1 (A), JPmiso2.1 (A), JPmiso3.1 (A)
- net C_MOSI: now also JPmosi1.2 (C), JPmosi2.2 (C), JPmosi3.2 (C); no longer JPmosi1.1 (A), JPmosi2.1 (A), JPmosi3.1 (A)
- net C_SCK: now also JPsck1.2 (C), JPsck2.2 (C), JPsck3.2 (C); no longer JPsck1.1 (A), JPsck2.1 (A), JPsck3.1 (A)
- net Electrode1: now also JPe1.1 (A), Rs1.1; no longer JPe1.2 (C), Rs11.1
- net Electrode10: now also JPe10.1 (A), Rs10.1; no longer JPe10.2 (C), Rs20.1
- net Electrode11: now also JPe11.1 (A), Rs11.1; no longer JPe11.2 (C), Rs21.1
- net Electrode12: now also JPe12.1 (A), Rs12.1; no longer JPe12.2 (C), Rs22.1
- net Electrode13: now also JPe13.1 (A), Rs13.1; no longer JPe13.2 (C), Rs23.1
- net Electrode14: now also JPe14.1 (A), Rs14.1; no longer JPe14.2 (C), Rs24.1
- net Electrode15: now also JPe15.1 (A), Rs15.1; no longer JPe15.2 (C), Rs25.1
- net Electrode16: now also JPe16.1 (A), Rs16.1; no longer JPe16.2 (C), Rs26.1
- net Electrode17: now also JPe17.1 (A), Rs17.1; no longer JPe17.2 (C), Rs27.1
- net Electrode18: now also JPe18.1 (A), Rs18.1; no longer JPe18.2 (C), Rs28.1
- net Electrode19: now also JPe19.1 (A), Rs19.1; no longer JPe19.2 (C), Rs29.1
- net Electrode2: now also JPe2.1 (A), Rs2.1; no longer JPe2.2 (C), Rs12.1
- net Electrode20: now also JPe20.1 (A), Rs20.1; no longer Rs30.1
- net Electrode21: now also JPe21.1 (A), Rs21.1; no longer JPe21.2 (C), Rs1.1
- net Electrode22: now also JPe22.1 (A), Rs22.1; no longer JPe22.2 (C), Rs2.1
- net Electrode23: now also JPe23.1 (A), Rs23.1; no longer JPe23.2 (C), Rs3.1
- net Electrode24: now also JPe24.1 (A), Rs24.1; no longer JPe24.2 (C), Rs4.1
- net Electrode25: now also JPe25.1 (A), Rs25.1; no longer JPe25.2 (C), Rs5.1
- net Electrode26: now also JPe26.1 (A), Rs26.1; no longer JPe26.2 (C), Rs6.1
- net Electrode27: now also JPe27.1 (A), Rs27.1; no longer JPe27.2 (C), Rs7.1
- net Electrode28: now also JPe28.1 (A), Rs28.1; no longer JPe28.2 (C), Rs8.1
- net Electrode29: now also JPe29.1 (A), Rs29.1; no longer JPe29.2 (C), Rs9.1
- net Electrode3: now also JPe3.1 (A), Rs3.1; no longer JPe3.2 (C), Rs13.1
- net Electrode30: now also JPe30.1 (A), Rs30.1; no longer JPe30.2 (C), Rs10.1
- net Electrode4: now also JPe4.1 (A), Rs4.1; no longer JPe4.2 (C), Rs14.1
- net Electrode5: now also JPe5.1 (A), Rs5.1; no longer JPe5.2 (C), Rs15.1
- net Electrode6: now also JPe6.1 (A), Rs6.1; no longer JPe6.2 (C), Rs16.1
- net Electrode7: now also JPe7.1 (A), Rs7.1; no longer JPe7.2 (C), Rs17.1
- net Electrode8: now also JPe8.1 (A), Rs8.1; no longer JPe8.2 (C), Rs18.1
- net Electrode9: now also JPe9.1 (A), Rs9.1; no longer JPe9.2 (C), Rs19.1
- net GND: now also H1.1, H2.1, H3.1, H4.1
- net MISO1: now also JPmiso1.1 (A); no longer JPmiso1.2 (C)
- net MISO2: now also JPmiso2.1 (A); no longer JPmiso2.2 (C)
- net MISO3: now also JPmiso3.1 (A); no longer JPmiso3.2 (C)
- net MOSI1: now also JPmosi1.1 (A); no longer JPmosi1.2 (C)
- net MOSI2: now also JPmosi2.1 (A); no longer JPmosi2.2 (C)
- net MOSI3: now also JPmosi3.1 (A); no longer JPmosi3.2 (C)
- net SCK1: now also JPsck1.1 (A); no longer JPsck1.2 (C)
- net SCK2: now also JPsck2.1 (A); no longer JPsck2.2 (C)
- net SCK3: now also JPsck3.1 (A); no longer JPsck3.2 (C)
- net at Cs1.1, U1.1 (SNS0K): now also Rs1.2; no longer Rs11.2
- net at Cs5.1, U1.11 (SNS4K): now also Rs5.2; no longer Rs15.2
- net at Cs6.1, U1.13 (SNS5K): now also Rs6.2; no longer Rs16.2
- net at Cs7.1, U1.19 (SNS6K): now also Rs7.2; no longer Rs17.2
- net at Cs8.1, U1.22 (DETECT0/SNS7K): now also Rs8.2; no longer Rs18.2
- net at Cs9.1, U1.25 (DETECT3/SNS8K): now also Rs9.2; no longer Rs19.2
- net at Cs10.1, U1.27 (DETECT5/SNS9K): now also Rs10.2; no longer Rs20.2
- net at Cs2.1, U1.3 (SNS1K): now also Rs2.2; no longer Rs12.2
- net at Cs3.1, U1.6 (SNS2K): now also Rs3.2; no longer Rs13.2
- net at Cs4.1, U1.9 (SNS3K): now also Rs4.2; no longer Rs14.2
- net at E11.1: now also JPe11.2 (C); no longer JPe11.1 (A)
- net at E12.1: now also JPe12.2 (C); no longer JPe12.1 (A)
- net at E13.1: now also JPe13.2 (C); no longer JPe13.1 (A)
- net at E14.1: now also JPe14.2 (C); no longer JPe14.1 (A)
- net at E15.1: now also JPe15.2 (C); no longer JPe15.1 (A)
- net at E16.1: now also JPe16.2 (C); no longer JPe16.1 (A)
- net at E17.1: now also JPe17.2 (C); no longer JPe17.1 (A)
- net at E18.1: now also JPe18.2 (C); no longer JPe18.1 (A)
- net at E19.1: now also JPe19.2 (C); no longer JPe19.1 (A)
- net at E20.1: now also JPe20.2 (C); no longer JPe20.1 (A)
- net at Cs11.1, U2.1 (SNS0K): now also Rs11.2; no longer Rs21.2
- net at Cs12.1, U2.3 (SNS1K): now also Rs12.2; no longer Rs22.2
- net at Cs13.1, U2.6 (SNS2K): now also Rs13.2; no longer Rs23.2
- net at Cs14.1, U2.9 (SNS3K): now also Rs14.2; no longer Rs24.2
- net at Cs15.1, U2.11 (SNS4K): now also Rs15.2; no longer Rs25.2
- net at Cs16.1, U2.13 (SNS5K): now also Rs16.2; no longer Rs26.2
- net at Cs17.1, U2.19 (SNS6K): now also Rs17.2; no longer Rs27.2
- net at Cs18.1, U2.22 (DETECT0/SNS7K): now also Rs18.2; no longer Rs28.2
- net at Cs19.1, U2.25 (DETECT3/SNS8K): now also Rs19.2; no longer Rs29.2
- net at Cs20.1, U2.27 (DETECT5/SNS9K): now also Rs20.2; no longer Rs30.2
- net at E30.1: now also JPe30.2 (C); no longer JPe30.1 (A)
- net at E29.1: now also JPe29.2 (C); no longer JPe29.1 (A)
- net at E28.1: now also JPe28.2 (C); no longer JPe28.1 (A)
- net at E27.1: now also JPe27.2 (C); no longer JPe27.1 (A)
- net at E26.1: now also JPe26.2 (C); no longer JPe26.1 (A)
- net at E25.1: now also JPe25.2 (C); no longer JPe25.1 (A)
- net at E24.1: now also JPe24.2 (C); no longer JPe24.1 (A)
- net at E23.1: now also JPe23.2 (C); no longer JPe23.1 (A)
- net at E22.1: now also JPe22.2 (C); no longer JPe22.1 (A)
- net at E21.1: now also JPe21.2 (C); no longer JPe21.1 (A)
- net at E10.1: now also JPe10.2 (C); no longer JPe10.1 (A)
- net at E9.1: now also JPe9.2 (C); no longer JPe9.1 (A)
- net at E8.1: now also JPe8.2 (C); no longer JPe8.1 (A)
- net at E7.1: now also JPe7.2 (C); no longer JPe7.1 (A)
- net at E6.1: now also JPe6.2 (C); no longer JPe6.1 (A)
- net at E5.1: now also JPe5.2 (C); no longer JPe5.1 (A)
- net at E4.1: now also JPe4.2 (C); no longer JPe4.1 (A)
- net at E3.1: now also JPe3.2 (C); no longer JPe3.1 (A)
- net at E2.1: now also JPe2.2 (C); no longer JPe2.1 (A)
- net at E1.1: now also JPe1.2 (C); no longer JPe1.1 (A)
- net at Cs21.1, U3.1 (SNS0K): now also Rs21.2; no longer Rs1.2
- net at Cs25.1, U3.11 (SNS4K): now also Rs25.2; no longer Rs5.2
- net at Cs26.1, U3.13 (SNS5K): now also Rs26.2; no longer Rs6.2
- net at Cs27.1, U3.19 (SNS6K): now also Rs27.2; no longer Rs7.2
- net at Cs28.1, U3.22 (DETECT0/SNS7K): now also Rs28.2; no longer Rs8.2
- net at Cs29.1, U3.25 (DETECT3/SNS8K): now also Rs29.2; no longer Rs9.2
- net at Cs30.1, U3.27 (DETECT5/SNS9K): now also Rs30.2; no longer Rs10.2
- net at Cs22.1, U3.3 (SNS1K): now also Rs22.2; no longer Rs2.2
- net at Cs23.1, U3.6 (SNS2K): now also Rs23.2; no longer Rs3.2
- net at Cs24.1, U3.9 (SNS3K): now also Rs24.2; no longer Rs4.2
Other:
- moved on the sheet: JPe1, JPe10, JPe11, JPe12, JPe13, JPe14, JPe15, JPe16, JPe17, JPe18, JPe19, JPe2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

Commit message: Layed out AT32QT1110
Parts:
- removed JPe1, JPe10, JPe11, JPe12, JPe13, JPe2, JPe3, JPe4, JPe5, JPe6, JPe7, JPe8, JPe9: Jumper_3_B12, Jumper:SolderJumper-3_P1.3mm_Bridged12_RoundedPad1.0x1.5mm_NumberLabels, symbol Jumper:SolderJumper_3_Bridged12
- added JPe? (x2): SolderJumper_3_Open, symbol Jumper:SolderJumper_3_Open
Changed lines of the file:
@@
 	6850 17350 6850 17550
-$Comp
-L Jumper:SolderJumper_3_Bridged12 JPe11
-U 1 1 6189BC90
-P 7050 15550
-F 0 "JPe11" V 7050 15600 50  0000 L CNN
-F 1 "Jumper_3_B12" V 7095 15618 50  0001 L CNN
-F 2 "Jumper:SolderJumper-3_P1.3mm_Bridged12_RoundedPad1.0x1.5mm_NumberLabels" H 7050 15550 50  0001 C CNN
-F 3 "~" H 7050 15550 50  0001 C CNN
-	1    7050 15550
-	-1   0    0    1
-$EndComp
-$Comp
-L Jumper:SolderJumper_3_Bridged12 JPe12
-U 1 1 618EC9AC
-P 7050 16000
-F 0 "JPe12" V 7050 16050 50  0000 L CNN
-F 1 "Jumper_3_B12" V 7095 16068 50  0001 L CNN
-F 2 "Jumper:SolderJumper-3_P1.3mm_Bridged12_RoundedPad1.0x1.5mm_NumberLabels" H 7050 16000 50  0001 C CNN
-F 3 "~" H 7050 16000 50  0001 C CNN
-	1    7050 16000
-	-1   0    0    1
-$EndComp
-$Comp
-L Jumper:SolderJumper_3_Bridged12 JPe13
-U 1 1 618FABEB
-P 7050 16450
-F 0 "JPe13" V 7050 16500 50  0000 L CNN
-F 1 "Jumper_3_B12" V 7095 16518 50  0001 L CNN
-F 2 "Jumper:SolderJumper-3_P1.3mm_Bridged12_RoundedPad1.0x1.5mm_NumberLabels" H 7050 16450 50  0001 C CNN
-F 3 "~" H 7050 16450 50  0001 C CNN
-	1    7050 16450
-	-1   0    0    1
-$EndComp
 $Comp
 L Jumper:SolderJumper_3_Bridged12 JPe14
@@
 Wire Wire Line
 	6650 12950 6450 12950
-$Comp
-L Jumper:SolderJumper_3_Bridged12 JPe9
-U 1 1 61F2ADDB
-P 7050 14100
-F 0 "JPe9" V 7050 14150 50  0000 L CNN
-F 1 "Jumper_3_B12" V 7095 14168 50  0001 L CNN
-F 2 "Jumper:SolderJumper-3_P1.3mm_Bridged12_RoundedPad1.0x1.5mm_NumberLabels" H 7050 14100 50  0001 C CNN
-F 3 "~" H 7050 14100 50  0001 C CNN
-	1    7050 14100
-	-1   0    0    1
-$EndComp
-$Comp
-L Jumper:SolderJumper_3_Bridged12 JPe8
-U 1 1 61F2ADED
-P 7050 13650
-F 0 "JPe8" V 7050 13700 50  0000 L CNN
-F 1 "Jumper_3_B12" V 7095 13718 50  0001 L CNN
-F 2 "Jumper:SolderJumper-3_P1.3mm_Bridged12_RoundedPad1.0x1.5mm_NumberLabels" H 7050 13650 50  0001 C CNN
-F 3 "~" H 7050 13650 50  0001 C CNN
-	1    7050 13650
-	-1   0    0    1
-$EndComp
-$Comp
-L Jumper:SolderJumper_3_Bridged12 JPe7
-U 1 1 61F2ADF3
-P 7050 13200
-F 0 "JPe7" V 7050 13250 50  0000 L CNN
-F 1 "Jumper_3_B12" V 7095 13268 50  0001 L CNN
-F 2 "Jumper:SolderJumper-3_P1.3mm_Bridged12_RoundedPad1.0x1.5mm_NumberLabels" H 7050 13200 50  0001 C CNN
-F 3 "~" H 7050 13200 50  0001 C CNN
-	1    7050 13200
-	-1   0    0    1
-$EndComp
-$Comp
-L Jumper:SolderJumper_3_Bridged12 JPe6
-U 1 1 61F2AE05
-P 7050 12750
-F 0 "JPe6" V 7050 12800 50  0000 L CNN
-F 1 "Jumper_3_B12" V 7095 12818 50  0001 L CNN
-F 2 "Jumper:SolderJumper-3_P1.3mm_Bridged12_RoundedPad1.0x1.5mm_NumberLabels" H 7050 12750 50  0001 C CNN
-F 3 "~" H 7050 12750 50  0001 C CNN
-	1    7050 12750
-	-1   0    0    1
-$EndComp
-$Comp
-L Jumper:SolderJumper_3_Bridged12 JPe5
-U 1 1 61F2AE0B
-P 7050 12250
-F 0 "JPe5" V 7050 12300 50  0000 L CNN
-F 1 "Jumper_3_B12" V 7095 12318 50  0001 L CNN
-F 2 "Jumper:SolderJumper-3_P1.3mm_Bridged12_RoundedPad1.0x1.5mm_NumberLabels" H 7050 12250 50  0001 C CNN
-F 3 "~" H 7050 12250 50  0001 C CNN
-	1    7050 12250
-	-1   0    0    1
-$EndComp
-$Comp
-L Jumper:SolderJumper_3_Bridged12 JPe4
-U 1 1 61F2AE1D
-P 7050 11800
-F 0 "JPe4" V 7050 11850 50  0000 L CNN
-F 1 "Jumper_3_B12" V 7095 11868 50  0001 L CNN
-F 2 "Jumper:SolderJumper-3_P1.3mm_Bridged12_RoundedPad1.0x1.5mm_NumberLabels" H 7050 11800 50  0001 C CNN
-F 3 "~" H 7050 11800 50  0001 C CNN
-	1    7050 11800
-	-1   0    0    1
-$EndComp
-$Comp
-L Jumper:SolderJumper_3_Bridged12 JPe3
-U 1 1 61F2AE23
-P 7050 11350
-F 0 "JPe3" V 7050 11400 50  0000 L CNN
-F 1 "Jumper_3_B12" V 7095 11418 50  0001 L CNN
-F 2 "Jumper:SolderJumper-3_P1.3mm_Bridged12_RoundedPad1.0x1.5mm_NumberLabels" H 7050 11350 50  0001 C CNN
-F 3 "~" H 7050 11350 50  0001 C CNN
-	1    7050 11350
-	-1   0    0    1
-$EndComp
-$Comp
-L Jumper:SolderJumper_3_Bridged12 JPe2
-U 1 1 61F2AE35
-P 7050 10900
-F 0 "JPe2" V 7050 10950 50  0000 L CNN
-F 1 "Jumper_3_B12" V 7095 10968 50  0001 L CNN
-F 2 "Jumper:SolderJumper-3_P1.3mm_Bridged12_RoundedPad1.0x1.5mm_NumberLabels" H 7050 10900 50  0001 C CNN
-F 3 "~" H 7050 10900 50  0001 C CNN
-	1    7050 10900
-	-1   0    0    1
-$EndComp
 Text Label 7250 12250 0    50   ~ 0
 Electrode5
@@
 Text Label 7250 10450 0    50   ~ 0
 Electrode1
-$Comp
-L Jumper:SolderJumper_3_Bridged12 JPe1
-U 1 1 61F2AE41
-P 7050 10450
-F 0 "JPe1" V 7050 10500 50  0000 L CNN
-F 1 "Jumper_3_B12" V 7095 10518 50  0001 L CNN
-F 2 "Jumper:SolderJumper-3_P1.3mm_Bridged12_RoundedPad1.0x1.5mm_NumberLabels" H 7050 10450 50  0001 C CNN
-F 3 "~" H 7050 10450 50  0001 C CNN
-	1    7050 10450
-	-1   0    0    1
-$EndComp
 Text Label 7250 14600 0    50   ~ 0
 Electrode10
-$Comp
-L Jumper:SolderJumper_3_Bridged12 JPe10
-U 1 1 61F2ADC9
-P 7050 14600
-F 0 "JPe10" V 7050 14650 50  0000 L CNN
-F 1 "Jumper_3_B12" V 7095 14668 50  0001 L CNN
-F 2 "Jumper:SolderJumper-3_P1.3mm_Bridged12_RoundedPad1.0x1.5mm_NumberLabels" H 7050 14600 50  0001 C CNN
-F 3 "~" H 7050 14600 50  0001 C CNN
-	1    7050 14600
-	-1   0    0    1
-$EndComp
 $Comp
 L Custom_Sensor_Touch:Electrode E10
@@
 	0    1    1    0
 $EndComp
+$Comp
+L Jumper:SolderJumper_3_Open JPe?
+U 1 1 63960F52
+P 7050 10450
+F 0 "JPe?" H 7050 10655 50  0000 C CNN
+F 1 "SolderJumper_3_Open" H 7050 10564 50  0000 C CNN
+F 2 "" H 7050 10450 50  0001 C CNN
+F 3 "~" H 7050 10450 50  0001 C CNN
+	1    7050 10450
+	-1   0    0    1
+$EndComp
+$Comp
+L Jumper:SolderJumper_3_Open JPe?
+U 1 1 639CAD31
+P 7050 10900
+F 0 "JPe?" H 7050 11105 50  0000 C CNN
+F 1 "SolderJumper_3_Open" H 7050 11014 50  0000 C CNN
+F 2 "" H 7050 10900 50  0001 C CNN
+F 3 "~" H 7050 10900 50  0001 C CNN
+	1    7050 10900
+	-1   0    0    1
+$EndComp
 $EndSCHEMATC
