File: pcbs/tinker/classical_guitar/classical_guitar_fretboard.sch (KiCad schematic (older format))
At the start: 160 parts, among them U1 AT42QT1110-A, U2 AT42QT1110-A, U3 AT42QT1110-A

Commit message: Replaced jumper pads
Parts:
- removed JPch1, JPch2, JPch3, JPe14, JPe15, JPe16, JPe17, JPe18, JPe19, JPe20, JPe21, JPe22, JPe23, JPe24, JPe25, JPe26, JPe27, JPe28, JPe29, JPe30, JPmiso1, JPmiso2, JPmiso3, JPmosi1, JPmosi2, JPmosi3, JPsck1, JPsck2, JPsck3: Jumper_3_B12, Jumper:SolderJumper-3_P1.3mm_Bridged12_RoundedPad1.0x1.5mm_NumberLabels, symbol Jumper:SolderJumper_3_Bridged12
- removed JPe? (x2): SolderJumper_3_Open, symbol Jumper:SolderJumper_3_Open
- added JPch1, JPch2, JPch3, JPe? (x30), JPmiso? (x3), JPmosi? (x3), JPsck? (x3): SolderJumper_3_Open, symbol Jumper:SolderJumper_3_Open

Commit message: Trace for 5-to-32 decoder before replacement with 4-to-16 decoder
Parts:
- removed Jdecoder_output1: Conn_02x16_Odd_Even, Connector_PinSocket_2.54mm:PinSocket_2x16_P2.54mm_Vertical, symbol Connector_Generic:Conn_02x16_Odd_Even
- added Jdecoder_output1: Conn_01x32, Connector_PinSocket_2.54mm:PinSocket_1x32_P2.54mm_Vertical, symbol Connector_Generic:Conn_01x32
- JPch1, JPch2, JPch3: footprint (none) -> Jumper:SolderJumper-3_P1.3mm_Open_RoundedPad1.0x1.5mm_NumberLabels
- JPe1, JPe10, JPe11, JPe12, JPe13, JPe14, JPe15, JPe16, JPe17, JPe18, JPe19, JPe2, JPe20, JPe21, JPe22, JPe23, JPe24, JPe25, JPe26, JPe27, JPe28, JPe29, JPe3, JPe30, JPe4, JPe5, JPe6, JPe7, JPe8, JPe9: renamed from JPe?; footprint (none) -> Jumper:SolderJumper-3_P1.3mm_Open_RoundedPad1.0x1.5mm_NumberLabels
- JPmiso1, JPmiso2, JPmiso3: renamed from JPmiso?; footprint (none) -> Jumper:SolderJumper-3_P1.3mm_Open_RoundedPad1.0x1.5mm_NumberLabels
- JPmosi1, JPmosi2, JPmosi3: renamed from JPmosi?; footprint (none) -> Jumper:SolderJumper-3_P1.3mm_Open_RoundedPad1.0x1.5mm_NumberLabels
- JPsck1, JPsck2, JPsck3: renamed from JPsck?; footprint (none) -> Jumper:SolderJumper-3_P1.3mm_Open_RoundedPad1.0x1.5mm_NumberLabels
Connections:
- net C_MISO: now also JPmiso1.1 (A), JPmiso2.1 (A), JPmiso3.1 (A); no longer JPmiso1.2 (C), JPmiso2.2 (C), JPmiso3.2 (C)
- net C_MOSI: now also JPmosi1.1 (A), JPmosi2.1 (A), JPmosi3.1 (A); no longer JPmosi1.2 (C), JPmosi2.2 (C), JPmosi3.2 (C)
- net C_SCK: now also JPsck1.1 (A), JPsck2.1 (A), JPsck3.1 (A); no longer JPsck1.2 (C), JPsck2.2 (C), JPsck3.2 (C)
- net Electrode1: now also JPe1.2 (C); no longer JPe1.1 (A)
- net Electrode10: now also JPe10.2 (C); no longer JPe10.1 (A)
- net Electrode11: now also JPe11.2 (C); no longer JPe11.1 (A)
- net Electrode12: now also JPe12.2 (C); no longer JPe12.1 (A)
- net Electrode13: now also JPe13.2 (C); no longer JPe13.1 (A)
- net Electrode14: now also JPe14.2 (C); no longer JPe14.1 (A)
- net Electrode15: now also JPe15.2 (C); no longer JPe15.1 (A)
- net Electrode16: now also JPe16.2 (C); no longer JPe16.1 (A)
- net Electrode17: now also JPe17.2 (C); no longer JPe17.1 (A)
- net Electrode18: now also JPe18.2 (C); no longer JPe18.1 (A)
- net Electrode19: now also JPe19.2 (C); no longer JPe19.1 (A)
- net Electrode2: now also JPe2.2 (C); no longer JPe2.1 (A)
- net Electrode20: now also JPe20.2 (C); no longer JPe20.1 (A)
- net Electrode21: now also JPe21.2 (C); no longer JPe21.1 (A)
- net Electrode22: now also JPe22.2 (C); no longer JPe22.1 (A)
- net Electrode23: now also JPe23.2 (C); no longer JPe23.1 (A)
- net Electrode24: now also JPe24.2 (C); no longer JPe24.1 (A)
- net Electrode25: now also JPe25.2 (C); no longer JPe25.1 (A)
- net Electrode26: now also JPe26.2 (C); no longer JPe26.1 (A)
- net Electrode27: now also JPe27.2 (C); no longer JPe27.1 (A)
- net Electrode28: now also JPe28.2 (C); no longer JPe28.1 (A)
- net Electrode29: now also JPe29.2 (C); no longer JPe29.1 (A)
- net Electrode3: now also JPe3.2 (C); no longer JPe3.1 (A)
- net Electrode30: now also JPe30.2 (C); no longer JPe30.1 (A)
- net Electrode4: now also JPe4.2 (C); no longer JPe4.1 (A)
- net Electrode5: now also JPe5.2 (C); no longer JPe5.1 (A)
- net Electrode6: now also JPe6.2 (C); no longer JPe6.1 (A)
- net Electrode7: now also JPe7.2 (C); no longer JPe7.1 (A)
- net Electrode8: now also JPe8.2 (C); no longer JPe8.1 (A)
- net Electrode9: now also JPe9.2 (C); no longer JPe9.1 (A)
- net MISO1: now also JPmiso1.2 (C); no longer JPmiso1.1 (A)
- net MISO2: now also JPmiso2.2 (C); no longer JPmiso2.1 (A)
- net MISO3: now also JPmiso3.2 (C); no longer JPmiso3.1 (A)
- net MOSI1: now also JPmosi1.2 (C); no longer JPmosi1.1 (A)
- net MOSI2: now also JPmosi2.2 (C); no longer JPmosi2.1 (A)
- net MOSI3: now also JPmosi3.2 (C); no longer JPmosi3.1 (A)
- net SCK1: now also JPsck1.2 (C); no longer JPsck1.1 (A)
- net SCK2: now also JPsck2.2 (C); no longer JPsck2.1 (A)
- net SCK3: now also JPsck3.2 (C); no longer JPsck3.1 (A)
- net at E10.1: now also JPe10.1 (A); no longer JPe10.2 (C)
- net at E9.1: now also JPe9.1 (A); no longer JPe9.2 (C)
- net at E7.1: now also JPe7.1 (A); no longer JPe7.2 (C)
- net at E6.1: now also JPe6.1 (A); no longer JPe6.2 (C)
- net at E8.1: now also JPe8.1 (A); no longer JPe8.2 (C)
- net at E5.1: now also JPe5.1 (A); no longer JPe5.2 (C)
- net at E4.1: now also JPe4.1 (A); no longer JPe4.2 (C)
- net at E3.1: now also JPe3.1 (A); no longer JPe3.2 (C)
- net at E2.1: now also JPe2.1 (A); no longer JPe2.2 (C)
- net at E1.1: now also JPe1.1 (A); no longer JPe1.2 (C)
- net at E30.1: now also JPe30.1 (A); no longer JPe30.2 (C)
- net at E29.1: now also JPe29.1 (A); no longer JPe29.2 (C)
- net at E27.1: now also JPe27.1 (A); no longer JPe27.2 (C)
- net at E26.1: now also JPe26.1 (A); no longer JPe26.2 (C)
- net at E28.1: now also JPe28.1 (A); no longer JPe28.2 (C)
- net at E25.1: now also JPe25.1 (A); no longer JPe25.2 (C)
- net at E24.1: now also JPe24.1 (A); no longer JPe24.2 (C)
- net at E23.1: now also JPe23.1 (A); no longer JPe23.2 (C)
- net at E22.1: now also JPe22.1 (A); no longer JPe22.2 (C)
- net at E21.1: now also JPe21.1 (A); no longer JPe21.2 (C)
- net at E20.1: now also JPe20.1 (A); no longer JPe20.2 (C)
- net at E19.1: now also JPe19.1 (A); no longer JPe19.2 (C)
- net at E17.1: now also JPe17.1 (A); no longer JPe17.2 (C)
- net at E16.1: now also JPe16.1 (A); no longer JPe16.2 (C)
- net at E18.1: now also JPe18.1 (A); no longer JPe18.2 (C)
- net at E15.1: now also JPe15.1 (A); no longer JPe15.2 (C)
- net at E14.1: now also JPe14.1 (A); no longer JPe14.2 (C)
- net at E13.1: now also JPe13.1 (A); no longer JPe13.2 (C)
- net at E12.1: now also JPe12.1 (A); no longer JPe12.2 (C)
- net at E11.1: now also JPe11.1 (A); no longer JPe11.2 (C)
- new net 5_to_32_decoder/~Y0: Jdecoder_output1.1 (Pin_1)
- new net 5_to_32_decoder/~Y1: Jdecoder_output1.2 (Pin_2)
- new net 5_to_32_decoder/~Y10: Jdecoder_output1.11 (Pin_11)
- new net 5_to_32_decoder/~Y11: Jdecoder_output1.12 (Pin_12)
- new net 5_to_32_decoder/~Y12: Jdecoder_output1.13 (Pin_13)
- new net 5_to_32_decoder/~Y13: Jdecoder_output1.14 (Pin_14)
- new net 5_to_32_decoder/~Y14: Jdecoder_output1.15 (Pin_15)
- new net 5_to_32_decoder/~Y15: Jdecoder_output1.16 (Pin_16)
- new net 5_to_32_decoder/~Y16: Jdecoder_output1.17 (Pin_17)
- new net 5_to_32_decoder/~Y17: Jdecoder_output1.18 (Pin_18)
- new net 5_to_32_decoder/~Y18: Jdecoder_output1.19 (Pin_19)
- new net 5_to_32_decoder/~Y19: Jdecoder_output1.20 (Pin_20)
- new net 5_to_32_decoder/~Y2: Jdecoder_output1.3 (Pin_3)
- new net 5_to_32_decoder/~Y20: Jdecoder_output1.21 (Pin_21)
- new net 5_to_32_decoder/~Y21: Jdecoder_output1.22 (Pin_22)
- new net 5_to_32_decoder/~Y22: Jdecoder_output1.23 (Pin_23)
- new net 5_to_32_decoder/~Y23: Jdecoder_output1.24 (Pin_24)
- new net 5_to_32_decoder/~Y24: Jdecoder_output1.25 (Pin_25)
- new net 5_to_32_decoder/~Y25: Jdecoder_output1.26 (Pin_26)
- new net 5_to_32_decoder/~Y26: Jdecoder_output1.27 (Pin_27)
- new net 5_to_32_decoder/~Y27: Jdecoder_output1.28 (Pin_28)
- new net 5_to_32_decoder/~Y28: Jdecoder_output1.29 (Pin_29)
- new net 5_to_32_decoder/~Y29: Jdecoder_output1.30 (Pin_30)
- new net 5_to_32_decoder/~Y3: Jdecoder_output1.4 (Pin_4)
- new net 5_to_32_decoder/~Y30: Jdecoder_output1.31 (Pin_31)
- new net 5_to_32_decoder/~Y31: Jdecoder_output1.32 (Pin_32)
- new net 5_to_32_decoder/~Y4: Jdecoder_output1.5 (Pin_5)
- new net 5_to_32_decoder/~Y5: Jdecoder_output1.6 (Pin_6)
- new net 5_to_32_decoder/~Y6: Jdecoder_output1.7 (Pin_7)
- new net 5_to_32_decoder/~Y7: Jdecoder_output1.8 (Pin_8)
- new net 5_to_32_decoder/~Y8: Jdecoder_output1.9 (Pin_9)
- new net 5_to_32_decoder/~Y9: Jdecoder_output1.10 (Pin_10)
Other:
- moved on the sheet: E1, E10, E11, E12, E13, E14, E15, E16, E17, E18, E19, E2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
