File: pcbs/tinker/classical_guitar/power_mp2359.sch (KiCad schematic (older format))
At the start: 18 parts, among them Q1 AO3401A, U4 MP2359

Commit message: Rearranging schematic
Parts:
- removed D3: YELLOW, LED_SMD:LED_0603_1608Metric, symbol Device:LED_Small
- removed R6: 1k5, Resistor_SMD:R_0603_1608Metric, symbol Device:R_Small
- U4: footprint (none) -> Package_TO_SOT_SMD:SOT-23-6_Handsoldering
Changed lines of the file:
@@
 Power Circuit\ncredits to Phil's Lab
-$Comp
-L Device:LED_Small D?
-U 1 1 61604297
-P 9150 5100
-AR Path="/615DF516/61604297" Ref="D?"  Part="1"
-AR Path="/615EFEC7/61604297" Ref="D?"  Part="1"
-AR Path="/61833101/61604297" Ref="D3"  Part="1"
-F 0 "D3" V 9196 5030 50  0000 R CNN
-F 1 "YELLOW" V 9105 5030 50  0000 R CNN
-F 2 "LED_SMD:LED_0603_1608Metric" V 9150 5100 50  0001 C CNN
-F 3 "~" V 9150 5100 50  0001 C CNN
-F 4 "C2286" H 9150 5100 50  0001 C CNN "LCSC Part #"
-	1    9150 5100
-	0    -1   -1   0
-$EndComp
-$Comp
-L Device:R_Small R?
-U 1 1 6160429E
-P 9150 5400
-AR Path="/615DF516/6160429E" Ref="R?"  Part="1"
-AR Path="/615EFEC7/6160429E" Ref="R?"  Part="1"
-AR Path="/61833101/6160429E" Ref="R6"  Part="1"
-F 0 "R6" H 9209 5446 50  0000 L CNN
-F 1 "1k5" H 9209 5355 50  0000 L CNN
-F 2 "Resistor_SMD:R_0603_1608Metric" H 9150 5400 50  0001 C CNN
-F 3 "~" H 9150 5400 50  0001 C CNN
-F 4 "C22843" H 9150 5400 50  0001 C CNN "LCSC Part #"
-	1    9150 5400
-	1    0    0    -1
-$EndComp
-Wire Wire Line
-	9150 5200 9150 5300
-Wire Wire Line
-	9150 5500 9150 5600
-Wire Wire Line
-	9150 4900 9150 5000
 $Comp
 L power:PWR_FLAG #FLG?
@@
 Text HLabel 7550 4600 1    50   Input ~ 0
 3V3
-Text HLabel 9150 4900 1    50   Input ~ 0
-3V3
 Text HLabel 4200 4950 3    50   Input ~ 0
 GND
@@
 GND
 Text HLabel 8850 3950 3    50   Input ~ 0
-GND
-Text HLabel 9150 5600 3    50   Input ~ 0
 GND
 Text HLabel 7550 5600 3    50   Input ~ 0
@@
 F 0 "U4" H 5850 3715 50  0000 C CNN
 F 1 "MP2359" H 5850 3624 50  0000 C CNN
-F 2 "" H 5850 3650 50  0001 C CNN
+F 2 "Package_TO_SOT_SMD:SOT-23-6_Handsoldering" H 5850 3650 50  0001 C CNN
 F 3 "" H 5850 3650 50  0001 C CNN
 	1    5850 3650

Commit message: Rearranged schematic again and establishing pcb layout
Parts:
- C1, C3, C4: footprint Capacitor_SMD:C_1206_3216Metric -> Capacitor_SMD:C_1206_3216Metric_Pad1.33x1.80mm_HandSolder
- C2: footprint Capacitor_SMD:C_0603_1608Metric -> Capacitor_SMD:C_0603_1608Metric_Pad1.08x0.95mm_HandSolder
Changed lines of the file:
@@
 F 0 "C1" H 4592 3546 50  0000 L CNN
 F 1 "10u" H 4592 3455 50  0000 L CNN
-F 2 "Capacitor_SMD:C_1206_3216Metric" H 4500 3500 50  0001 C CNN
+F 2 "Capacitor_SMD:C_1206_3216Metric_Pad1.33x1.80mm_HandSolder" H 4500 3500 50  0001 C CNN
 F 3 "~" H 4500 3500 50  0001 C CNN
 F 4 "C13585" H 4500 3500 50  0001 C CNN "LCSC Part #"
@@
 F 0 "C3" H 8592 3896 50  0000 L CNN
 F 1 "10uF" H 8592 3805 50  0000 L CNN
-F 2 "Capacitor_SMD:C_1206_3216Metric" H 8500 3850 50  0001 C CNN
+F 2 "Capacitor_SMD:C_1206_3216Metric_Pad1.33x1.80mm_HandSolder" H 8500 3850 50  0001 C CNN
 F 3 "~" H 8500 3850 50  0001 C CNN
 F 4 "C13585" H 8500 3850 50  0001 C CNN "LCSC Part #"
@@
 F 0 "C2" H 7442 3146 50  0000 L CNN
 F 1 "10nF" H 7442 3055 50  0000 L CNN
-F 2 "Capacitor_SMD:C_0603_1608Metric" H 7350 3100 50  0001 C CNN
+F 2 "Capacitor_SMD:C_0603_1608Metric_Pad1.08x0.95mm_HandSolder" H 7350 3100 50  0001 C CNN
 F 3 "~" H 7350 3100 50  0001 C CNN
 F 4 "C57112" H 7350 3100 50  0001 C CNN "LCSC Part #"
@@
 F 0 "C4" H 8942 3896 50  0000 L CNN
 F 1 "10uF" H 8942 3805 50  0000 L CNN
-F 2 "Capacitor_SMD:C_1206_3216Metric" H 8850 3850 50  0001 C CNN
+F 2 "Capacitor_SMD:C_1206_3216Metric_Pad1.33x1.80mm_HandSolder" H 8850 3850 50  0001 C CNN
 F 3 "~" H 8850 3850 50  0001 C CNN
 F 4 "C13585" H 8850 3850 50  0001 C CNN "LCSC Part #"
